File: pcb/bpf/bpf.kicad_sch (KiCad schematic)
At the start: 21 parts, among them J1 input, J2 power_input, J3 audio_out, U1 TI080, U2 TI080

Commit message: finalize layout and routing
Parts:
- added C1, C2: 1uF, Capacitor_THT:CP_Radial_D5.0mm_P2.00mm, symbol Device:C_Polarized_Small_US
- C3: renamed from C1; footprint Capacitor_THT:C_Disc_D7.5mm_W5.0mm_P7.50mm -> Capacitor_THT:C_Disc_D5.0mm_W2.5mm_P5.00mm
- C4: renamed from C2; footprint Capacitor_THT:C_Disc_D7.5mm_W5.0mm_P7.50mm -> Capacitor_THT:C_Disc_D5.0mm_W2.5mm_P5.00mm
- C5: renamed from C3; footprint Capacitor_THT:C_Disc_D7.5mm_W5.0mm_P7.50mm -> Capacitor_THT:C_Disc_D5.0mm_W2.5mm_P5.00mm
- C6: renamed from C4; footprint Capacitor_THT:C_Disc_D7.5mm_W5.0mm_P7.50mm -> Capacitor_THT:C_Disc_D5.0mm_W2.5mm_P5.00mm
- R1: value 22k ohms -> 22k
- R2, R5, R6: value 11k ohms -> 11k
Connections:
- net +5V: now also C2.1
- net -5V: now also C1.2
- net GND: now also R4.2, C1.1, C2.2; no longer R4.1
- net at D2.2 (A): now also R4.1; no longer R4.2
Other:
- moved on the sheet: R4
